Commit message: [BUILD] - Build robot

File: src/anhc_robot_description/urdf/control/anhc_control.xacro (robot description, xacro)
@@ -10,5 +10,5 @@
         <plugin>gz_ros2_control/GazeboSimSystem</plugin>
       </hardware>
-      <joint name="anhc_fl_wheel_joint">
+      <joint name="front_left_wheel_joint">
         <command_interface name="velocity">
           <param name="min">-5.0</param>
@@ -18,5 +18,5 @@
         <state_interface name="velocity"/>
       </joint>
-      <joint name="anhc_fr_wheel_joint">
+      <joint name="front_right_wheel_joint">
         <command_interface name="velocity">
           <param name="min">-5.0</param>
@@ -26,5 +26,5 @@
         <state_interface name="velocity"/>
       </joint>
-      <joint name="anhc_rl_wheel_joint">
+      <joint name="back_left_wheel_joint">
         <command_interface name="velocity">
           <param name="min">-5.0</param>
@@ -34,5 +34,5 @@
         <state_interface name="velocity"/>
       </joint>
-      <joint name="anhc_rr_wheel_joint">
+      <joint name="back_right_wheel_joint">
         <command_interface name="velocity">
           <param name="min">-5.0</param>
@@ -62,10 +62,10 @@
         filename="gz-sim-diff-drive-system"
         name="gz::sim::systems::DiffDrive">
-        <left_joint>anhc_fl_wheel_joint</left_joint>
-        <left_joint>anhc_rl_wheel_joint</left_joint>
-        <right_joint>anhc_fr_wheel_joint</right_joint>
-        <right_joint>anhc_rr_wheel_joint</right_joint>
-        <wheel_separation>0.400</wheel_separation>
-        <wheel_radius>0.075</wheel_radius>
+        <left_joint>front_left_wheel_joint</left_joint>
+        <left_joint>back_left_wheel_joint</left_joint>
+        <right_joint>front_right_wheel_joint</right_joint>
+        <right_joint>back_right_wheel_joint</right_joint>
+        <wheel_separation>0.169</wheel_separation>
+        <wheel_radius>0.0325</wheel_radius>
         <!-- Listen for velocity commands -->
         <topic>/anhc/cmd_vel</topic>

File: src/anhc_robot_description/urdf/mech/anhc_base.xacro (robot description, xacro)
@@ -1,63 +1,27 @@
 <?xml version="1.0"?>
 <robot xmlns:xacro="http://www.ros.org/wiki/xacro">
-  <!-- ═══════════════════════════════════════════════════════════
-       ANHC BASE MECHANICAL DESCRIPTION
-       Defines: chassis, 4 wheels, caster (base_footprint → base_link)
-       Coordinate convention: X=forward, Y=left, Z=up
-       ═══════════════════════════════════════════════════════════ -->
-  <!-- ── Tunable Parameters ─────────────────────────────────── -->
-  <xacro:property name="base_length"    value="0.50"/>   <!-- meters -->
-  <xacro:property name="base_width"     value="0.35"/>
-  <xacro:property name="base_height"    value="0.15"/>
-  <xacro:property name="base_mass"      value="10.0"/>   <!-- kg     -->
-  <xacro:property name="wheel_radius"   value="0.075"/>
-  <xacro:property name="wheel_width"    value="0.05"/>
-  <xacro:property name="wheel_mass"     value="0.5"/>
-  <!-- Wheel X offset from center (front/rear) -->
-  <xacro:property name="wheel_x_offset" value="0.175"/>
-  <!-- Wheel Y offset from center (left/right) -->
-  <xacro:property name="wheel_y_offset" value="0.200"/>
-  <!-- Wheel Z = radius (sits on ground) minus half base height -->
-  <xacro:property name="wheel_z_offset" value="0.0"/>
-  <!-- ── Inertia Macros ──────────────────────────────────────── -->
-  <!-- Box inertia (chassis) -->
-  <xacro:macro name="box_inertia" params="m l w h">
-    <inertial>
-      <mass value="${m}"/>
-      <inertia
-        ixx="${(m/12.0)*(w*w + h*h)}"  ixy="0" ixz="0"
-        iyy="${(m/12.0)*(l*l + h*h)}"  iyz="0"
-        izz="${(m/12.0)*(l*l + w*w)}"/>
-    </inertial>
-  </xacro:macro>
-  <!-- Cylinder inertia (wheels) -->
-  <xacro:macro name="cylinder_inertia" params="m r h">
-    <inertial>
-      <mass value="${m}"/>
-      <inertia
-        ixx="${(m/12.0)*(3*r*r + h*h)}"  ixy="0" ixz="0"
-        iyy="${(m/12.0)*(3*r*r + h*h)}"  iyz="0"
-        izz="${(m/2.0)*r*r}"/>
-    </inertial>
-  </xacro:macro>
-  <!-- ── Wheel Macro ─────────────────────────────────────────── -->
-  <!--
-    Creates one wheel link + joint.
-    Parameters:
-      prefix  : fl | fr | rl | rr
-      x_sign  : +1 (front) | -1 (rear)
-      y_sign  : +1 (left)  | -1 (right)
-  -->
-  <xacro:macro name="anhc_wheel" params="prefix x_sign y_sign">
-    <!-- Link -->
-    <link name="anhc_${prefix}_wheel_link">
+  <!-- Rosmaster X3 dimensions -->
+  <xacro:property name="total_width" value="0.19940"/>
+  <xacro:property name="wheel_width" value="0.0304"/>
+  <xacro:property name="wheel_radius" value="0.0325"/>
+  <xacro:property name="total_height" value="0.26225"/>
+  <xacro:property name="base_length" value="0.300"/>
+  <xacro:property name="centered_length" value="0.238"/>
+  <xacro:property name="base_x_offset" value="${(centered_length - base_length) / 2}"/>
+  <xacro:property name="base_size_x" value="${base_length}"/>
+  <xacro:property name="base_size_y" value="${total_width - (2 * wheel_width)}"/>
+  <xacro:property name="base_size_z" value="${total_height - (2 * wheel_radius)}"/>
+  <xacro:property name="base_mass" value="4.6"/>
+  <xacro:property name="wheel_mass" value="0.091"/>
+  <xacro:property name="wheel_xoff" value="0.08"/>
+  <xacro:property name="wheel_yoff" value="-0.01"/>
+  <xacro:property name="wheel_separation" value="0.169"/>
+  <xacro:macro name="rosmaster_wheel" params="side joint_name x_reflect y_reflect mesh_name">
+    <link name="${side}_wheel_link">
       <visual>
         <origin xyz="0 0 0" rpy="${pi/2} 0 0"/>
         <geometry>
-          <cylinder radius="${wheel_radius}" length="${wheel_width}"/>
+          <mesh filename="file://$(find anhc_robot_description)/meshes/rosmaster_x3/visual/${mesh_name}"/>
         </geometry>
-        <material name="anhc_wheel_material">
-          <color rgba="0.1 0.1 0.1 1.0"/>
-        </material>
       </visual>
       <collision>
@@ -67,57 +31,55 @@
         </geometry>
       </collision>
-      <xacro:cylinder_inertia m="${wheel_mass}" r="${wheel_radius}" h="${wheel_width}"/>
+      <inertial>
+        <origin xyz="0 0 0" rpy="0 0 0"/>
+        <mass value="${wheel_mass}"/>
+        <inertia
+          ixx="${(wheel_mass/12.0) * (3*wheel_radius*wheel_radius + wheel_width*wheel_width)}" ixy="0" ixz="0"
+          iyy="${(wheel_mass/2.0) * (wheel_radius*wheel_radius)}" iyz="0"
+          izz="${(wheel_mass/12.0) * (3*wheel_radius*wheel_radius + wheel_width*wheel_width)}"/>
+      </inertial>
     </link>
-    <!-- Continuous Joint (wheel spins freely around Y axis) -->
-    <joint name="anhc_${prefix}_wheel_joint" type="continuous">
-      <parent link="anhc_base_link"/>
-      <child  link="anhc_${prefix}_wheel_link"/>
-      <origin
-        xyz="${x_sign * wheel_x_offset}
-             ${y_sign * wheel_y_offset}
-             ${wheel_z_offset}"
-        rpy="0 0 0"/>
+    <joint name="${joint_name}" type="continuous">
       <axis xyz="0 1 0"/>
-      <dynamics damping="0.1" friction="0.1"/>
-      <limit effort="10.0" velocity="5.0"/>
+      <parent link="base_link"/>
+      <child link="${side}_wheel_link"/>
+      <origin xyz="${x_reflect*wheel_xoff} ${y_reflect*(wheel_separation/2+wheel_yoff)} ${-wheel_radius}" rpy="0 0 0"/>
     </joint>
+    <gazebo reference="${side}_wheel_link">
+      <mu1>1.0</mu1>
+      <mu2>0.0</mu2>
+    </gazebo>
   </xacro:macro>
-  <!-- ══════════════════════════════════════════════════════════
-       LINKS
-       ══════════════════════════════════════════════════════════ -->
-  <!-- base_footprint: virtual link at ground level, origin of the robot -->
   <link name="base_footprint"/>
-  <!-- base_link: geometric center of chassis, elevated above ground -->
-  <link name="anhc_base_link">
+  <link name="base_link">
     <visual>
+      <geometry>
+        <mesh filename="file://$(find anhc_robot_description)/meshes/rosmaster_x3/visual/base_link_X3.STL"/>
+      </geometry>
       <origin xyz="0 0 0" rpy="0 0 0"/>
-      <geometry>
-        <box size="${base_length} ${base_width} ${base_height}"/>
-      </geometry>
-      <material name="anhc_chassis_material">
-        <color rgba="0.2 0.5 0.8 1.0"/>
-      </material>
     </visual>
     <collision>
-      <origin xyz="0 0 0" rpy="0 0 0"/>
       <geometry>
-        <box size="${base_length} ${base_width} ${base_height}"/>
+        <box size="${base_size_x} ${base_size_y} ${base_size_z}"/>
       </geometry>
+      <origin xyz="${base_x_offset} 0 ${base_size_z/2 + wheel_radius/4}" rpy="0 0 0"/>
     </collision>
-    <xacro:box_inertia m="${base_mass}" l="${base_length}" w="${base_width}" h="${base_height}"/>
+    <inertial>
+      <origin xyz="${base_x_offset} 0 ${base_size_z/2 + wheel_radius/4}" rpy="0 0 0"/>
+      <mass value="${base_mass}"/>
+      <inertia
+        ixx="${(1/12) * base_mass * ((base_size_y * base_size_y) + (base_size_z * base_size_z))}" ixy="0.0" ixz="0.0"
+        iyy="${(1/12) * base_mass * ((base_size_x * base_size_x) + (base_size_z * base_size_z))}" iyz="0.0"
+        izz="${(1/12) * base_mass * ((base_size_x * base_size_x) + (base_size_y * base_size_y))}"/>
+    </inertial>
   </link>
-  <!-- ══════════════════════════════════════════════════════════
-       JOINTS
-       ══════════════════════════════════════════════════════════ -->
-  <!-- base_footprint → base_link: lift chassis off the ground by wheel_radius -->
-  <joint name="base_footprint_joint" type="fixed">
+  <joint name="base_joint" type="fixed">
     <parent link="base_footprint"/>
-    <child  link="anhc_base_link"/>
+    <child link="base_link"/>
     <origin xyz="0 0 ${wheel_radius}" rpy="0 0 0"/>
   </joint>
-  <!-- ── Instantiate 4 Wheels ────────────────────────────────── -->
-  <!-- Front-Left  --> <xacro:anhc_wheel prefix="fl" x_sign=" 1" y_sign=" 1"/>
-  <!-- Front-Right --> <xacro:anhc_wheel prefix="fr" x_sign=" 1" y_sign="-1"/>
-  <!-- Rear-Left   --> <xacro:anhc_wheel prefix="rl" x_sign="-1" y_sign=" 1"/>
-  <!-- Rear-Right  --> <xacro:anhc_wheel prefix="rr" x_sign="-1" y_sign="-1"/>
+  <xacro:rosmaster_wheel side="front_left"  joint_name="front_left_wheel_joint"  x_reflect=" 1" y_reflect=" 1" mesh_name="front_left_wheel_X3.STL"/>
+  <xacro:rosmaster_wheel side="front_right" joint_name="front_right_wheel_joint" x_reflect=" 1" y_reflect="-1" mesh_name="front_right_wheel_X3.STL"/>
+  <xacro:rosmaster_wheel side="back_left"   joint_name="back_left_wheel_joint"   x_reflect="-1" y_reflect=" 1" mesh_name="back_left_wheel_X3.STL"/>
+  <xacro:rosmaster_wheel side="back_right"  joint_name="back_right_wheel_joint"  x_reflect="-1" y_reflect="-1" mesh_name="back_right_wheel_X3.STL"/>
 </robot>

File: src/anhc_robot_description/urdf/robots/anhc_robot.xacro (robot description, xacro)
@@ -18,5 +18,5 @@
   <material name="anhc_camera_material">  <color rgba="0.1 0.1 0.1 1.0"/> </material>
   <!-- ── Instantiate Mechanical Base ─────────────────────────── -->
-  <!-- (base.xacro defines base_footprint, anhc_base_link, 4 wheels) -->
+  <!-- (base.xacro defines base_footprint, base_link, 4 wheels) -->
   <!-- ── Place 3D LiDAR on top-center of chassis ─────────────── -->
   <!--
@@ -26,5 +26,5 @@
   -->
   <xacro:anhc_lidar_3d
-    parent_link="anhc_base_link"
+    parent_link="base_link"
     xyz="0.0 0.0 0.110"
     rpy="0 0 0"/>
@@ -35,5 +35,5 @@
   -->
   <xacro:anhc_lidar_2d
-    parent_link="anhc_base_link"
+    parent_link="base_link"
     xyz="0.20 0.0 0.095"
     rpy="0 0 0"/>
@@ -45,5 +45,5 @@
   -->
   <xacro:anhc_camera
-    parent_link="anhc_base_link"
+    parent_link="base_link"
     xyz="0.225 0.0 0.10"
     rpy="0 0 0"/>
@@ -60,10 +60,10 @@
   </link>
   <joint name="anhc_imu_joint" type="fixed">
-    <parent link="anhc_base_link"/>
+    <parent link="base_link"/>
     <child  link="anhc_imu_link"/>
     <origin xyz="0 0 0" rpy="0 0 0"/>
   </joint>
   <!-- ── Gazebo Physics Properties ────────────────────────────── -->
-  <gazebo reference="anhc_base_link">
+  <gazebo reference="base_link">
     <mu1>0.8</mu1>
     <mu2>0.8</mu2>
@@ -72,17 +72,17 @@
     <material>Gazebo/Blue</material>
   </gazebo>
-  <gazebo reference="anhc_fl_wheel_link">
+  <gazebo reference="front_left_wheel_link">
     <mu1>1.0</mu1><mu2>1.0</mu2><kp>1e6</kp><kd>1.0</kd>
     <material>Gazebo/Black</material>
   </gazebo>
-  <gazebo reference="anhc_fr_wheel_link">
+  <gazebo reference="front_right_wheel_link">
     <mu1>1.0</mu1><mu2>1.0</mu2><kp>1e6</kp><kd>1.0</kd>
     <material>Gazebo/Black</material>
   </gazebo>
-  <gazebo reference="anhc_rl_wheel_link">
+  <gazebo reference="back_left_wheel_link">
     <mu1>1.0</mu1><mu2>1.0</mu2><kp>1e6</kp><kd>1.0</kd>
     <material>Gazebo/Black</material>
   </gazebo>
-  <gazebo reference="anhc_rr_wheel_link">
+  <gazebo reference="back_right_wheel_link">
     <mu1>1.0</mu1><mu2>1.0</mu2><kp>1e6</kp><kd>1.0</kd>
     <material>Gazebo/Black</material>

File: src/anhc_robot_description/urdf/sensors/anhc_camera.xacro (robot description, xacro)
@@ -2,11 +2,9 @@
 <robot xmlns:xacro="http://www.ros.org/wiki/xacro">
   <xacro:macro name="anhc_camera" params="parent_link xyz rpy">
-    <link name="anhc_camera_link">
+    <link name="camera_link">
       <visual>
+        <!-- Use simple box to avoid mesh local-frame offsets -->
         <origin xyz="0 0 0" rpy="0 0 0"/>
         <geometry><box size="0.025 0.09 0.025"/></geometry>
-        <material name="anhc_camera_material">
-          <color rgba="0.1 0.1 0.1 1.0"/>
-        </material>
       </visual>
       <collision>
@@ -20,21 +18,21 @@
       </inertial>
     </link>
-    <joint name="anhc_camera_joint" type="fixed">
+    <joint name="camera_joint" type="fixed">
       <parent link="${parent_link}"/>
-      <child  link="anhc_camera_link"/>
+      <child  link="camera_link"/>
       <origin xyz="${xyz}" rpy="${rpy}"/>
     </joint>
-    <link name="anhc_camera_optical_link"/>
-    <joint name="anhc_camera_optical_joint" type="fixed">
-      <parent link="anhc_camera_link"/>
-      <child  link="anhc_camera_optical_link"/>
+    <link name="camera_optical_link"/>
+    <joint name="camera_optical_joint" type="fixed">
+      <parent link="camera_link"/>
+      <child  link="camera_optical_link"/>
       <origin xyz="0 0 0" rpy="${-pi/2} 0 ${-pi/2}"/>
     </joint>
-    <gazebo reference="anhc_camera_link">
+    <gazebo reference="camera_link">
       <sensor name="anhc_camera_sensor" type="camera">
-        <topic>/anhc/camera</topic>
+        <topic>/anhc/camera/image</topic>
+        <frame_id>camera_optical_link</frame_id>
         <update_rate>30</update_rate>
         <always_on>true</always_on>
-        <enabled>true</enabled>
         <visualize>false</visualize>
         <camera>

File: src/anhc_robot_description/urdf/sensors/anhc_lidar_2d.xacro (robot description, xacro)
@@ -2,41 +2,46 @@
 <robot xmlns:xacro="http://www.ros.org/wiki/xacro">
   <xacro:macro name="anhc_lidar_2d" params="parent_link xyz rpy">
-    <link name="anhc_lidar_2d_link">
+    <link name="laser_frame">
       <visual>
-        <origin xyz="0 0 0" rpy="0 0 0"/>
-        <geometry><box size="0.07 0.07 0.04"/></geometry>
-        <material name="anhc_lidar2d_material">
-          <color rgba="0.1 0.8 0.1 1.0"/>
-        </material>
+        <origin xyz="0 0 0" rpy="${-pi/2} 0 0"/>
+        <geometry>
+          <mesh filename="file://$(find anhc_robot_description)/meshes/rplidar/rplidar_s2.stl" scale="0.001 0.001 0.001"/>
+        </geometry>
       </visual>
       <collision>
         <origin xyz="0 0 0" rpy="0 0 0"/>
-        <geometry><box size="0.07 0.07 0.04"/></geometry>
+        <geometry><cylinder radius="0.0385" length="0.0398"/></geometry>
       </collision>
       <inertial>
-        <mass value="0.05"/>
-        <inertia ixx="0.001" ixy="0" ixz="0"
-                 iyy="0.001" iyz="0" izz="0.001"/>
+        <mass value="0.185"/>
+        <inertia ixx="0.000128" ixy="0" ixz="0"
+                 iyy="0.000128" iyz="0" izz="0.000659"/>
       </inertial>
     </link>
     <joint name="anhc_lidar_2d_joint" type="fixed">
       <parent link="${parent_link}"/>
-      <child  link="anhc_lidar_2d_link"/>
+      <child  link="laser_frame"/>
       <origin xyz="${xyz}" rpy="${rpy}"/>
     </joint>
-    <gazebo reference="anhc_lidar_2d_link">
+    <!--
+      Gazebo Harmonic: sensor MUST be inside <gazebo reference="link_name">
+      AND world must have gz-sim-sensors-system plugin loaded.
+      type="gpu_lidar" requires ogre2 render engine.
+    -->
+    <gazebo reference="laser_frame">
       <sensor name="anhc_lidar_2d_sensor" type="gpu_lidar">
+        <pose>0 0 0 0 0 0</pose>
         <topic>/anhc/scan</topic>
-        <update_rate>15</update_rate>
+        <frame_id>laser_frame</frame_id>
+        <update_rate>10</update_rate>
         <always_on>true</always_on>
-        <enabled>true</enabled>
-        <visualize>true</visualize>
-        <lidar>
+        <visualize>false</visualize>
+        <ray>
           <scan>
             <horizontal>
-              <samples>540</samples>
+              <samples>720</samples>
               <resolution>1</resolution>
-              <min_angle>-2.35619</min_angle>
-              <max_angle>2.35619</max_angle>
+              <min_angle>-3.14159</min_angle>
+              <max_angle>3.14159</max_angle>
             </horizontal>
             <vertical>
@@ -48,14 +53,9 @@
           </scan>
           <range>
-            <min>0.1</min>
+            <min>0.20</min>
             <max>30.0</max>
-            <resolution>0.01</resolution>
+            <resolution>0.013</resolution>
           </range>
-          <noise>
-            <type>gaussian</type>
-            <mean>0.0</mean>
-            <stddev>0.005</stddev>
-          </noise>
-        </lidar>
+        </ray>
       </sensor>
     </gazebo>

File: src/anhc_robot_description/urdf/sensors/anhc_lidar_3d.xacro (robot description, xacro)
@@ -6,5 +6,5 @@
         <origin xyz="0 0 0" rpy="0 0 0"/>
         <geometry><cylinder radius="0.04" length="0.07"/></geometry>
-        <material name="anhc_lidar_material">
+        <material name="anhc_lidar3d_mat">
           <color rgba="0.8 0.1 0.1 1.0"/>
         </material>
@@ -27,8 +27,9 @@
     <gazebo reference="anhc_lidar_3d_link">
       <sensor name="anhc_lidar_3d_sensor" type="gpu_lidar">
+        <pose>0 0 0 0 0 0</pose>
         <topic>/anhc/lidar_3d/points</topic>
+        <frame_id>anhc_lidar_3d_link</frame_id>
         <update_rate>10</update_rate>
         <always_on>true</always_on>
-        <enabled>true</enabled>
         <visualize>false</visualize>
         <lidar>
@@ -37,6 +38,6 @@
               <samples>360</samples>
               <resolution>1</resolution>
-              <min_angle>-3.14159</min_angle>
-              <max_angle>3.14159</max_angle>
+              <min_angle>-3.14159265</min_angle>
+              <max_angle>3.14159265</max_angle>
             </horizontal>
             <vertical>
