Commit message: [FIX]- Fix position lidar and camera

File: src/anhc_robot_description/urdf/robots/anhc_robot.xacro (robot description, xacro)
@@ -7,5 +7,4 @@
   <!-- ── Include subsystem xacros ────────────────────────────── -->
   <xacro:include filename="$(find anhc_robot_description)/urdf/mech/anhc_base.xacro"/>
-  <xacro:include filename="$(find anhc_robot_description)/urdf/sensors/anhc_lidar_3d.xacro"/>
   <xacro:include filename="$(find anhc_robot_description)/urdf/sensors/anhc_lidar_2d.xacro"/>
   <xacro:include filename="$(find anhc_robot_description)/urdf/sensors/anhc_camera.xacro"/>
@@ -19,32 +18,15 @@
   <!-- ── Instantiate Mechanical Base ─────────────────────────── -->
   <!-- (base.xacro defines base_footprint, base_link, 4 wheels) -->
-  <!-- ── Place 3D LiDAR on top-center of chassis ─────────────── -->
-  <!--
-    base_height/2 = 0.075  → top surface of chassis
-    lidar cylinder height/2 = 0.035
-    Total z = 0.075 + 0.035 = 0.110
-  -->
-  <xacro:anhc_lidar_3d
-    parent_link="base_link"
-    xyz="0.0 0.0 0.110"
-    rpy="0 0 0"/>
-  <!-- ── Place 2D LiDAR at front of chassis ───────────────────── -->
-  <!--
-    x = base_length/2 = 0.25 (front edge)
-    z = base_height/2 + lidar_box_height/2 = 0.075 + 0.02 = 0.095
-  -->
+  <!-- 3D LiDAR is disabled for the old robot profile -->
+  <!-- ── Place 2D LiDAR on top-front of chassis ───────────────── -->
+  <!-- Tuned to stay visually attached to the body mesh -->
   <xacro:anhc_lidar_2d
     parent_link="base_link"
-    xyz="0.20 0.0 0.095"
+    xyz="0.03 0.0 0.08"
     rpy="0 0 0"/>
-  <!-- ── Place RGB Camera at front, slightly raised ────────────── -->
-  <!--
-    x = 0.225 (just at front edge)
-    z = 0.10 (above chassis top)
-    pitch = 0 (looking straight forward)
-  -->
+  <!-- ── Place RGB Camera on top-front, near LiDAR ────────────── -->
   <xacro:anhc_camera
     parent_link="base_link"
-    xyz="0.225 0.0 0.10"
+    xyz="0.14 0.0 0.05"
     rpy="0 0 0"/>
   <!-- ── Instantiate ros2_control + Gazebo plugins ────────────── -->

File: src/anhc_robot_description/urdf/sensors/anhc_camera.xacro (robot description, xacro)
@@ -4,7 +4,9 @@
     <link name="camera_link">
       <visual>
-        <!-- Use simple box to avoid mesh local-frame offsets -->
-        <origin xyz="0 0 0" rpy="0 0 0"/>
-        <geometry><box size="0.025 0.09 0.025"/></geometry>
+        <!-- Original D435 mesh with corrected local orientation -->
+        <origin xyz="0 0 0" rpy="${pi/2} 0 ${pi/2}"/>
+        <geometry>
+          <mesh filename="file://$(find anhc_robot_description)/meshes/intel_realsense/visual/d435.stl"/>
+        </geometry>
       </visual>
       <collision>

File: src/anhc_robot_description/urdf/sensors/anhc_lidar_2d.xacro (robot description, xacro)
@@ -4,8 +4,12 @@
     <link name="laser_frame">
       <visual>
+        <!-- Original RPLidar mesh, rotated to match ROS X-forward convention -->
         <origin xyz="0 0 0" rpy="${-pi/2} 0 0"/>
         <geometry>
           <mesh filename="file://$(find anhc_robot_description)/meshes/rplidar/rplidar_s2.stl" scale="0.001 0.001 0.001"/>
         </geometry>
+        <material name="anhc_lidar2d_mat">
+          <color rgba="0.1 0.1 0.1 1.0"/>
+        </material>
       </visual>
       <collision>
@@ -30,5 +34,5 @@
     -->
     <gazebo reference="laser_frame">
-      <sensor name="anhc_lidar_2d_sensor" type="gpu_lidar">
+      <sensor name="anhc_lidar_2d_sensor" type="lidar">
         <pose>0 0 0 0 0 0</pose>
         <topic>/anhc/scan</topic>
@@ -40,5 +44,5 @@
           <scan>
             <horizontal>
-              <samples>720</samples>
+              <samples>360</samples>
               <resolution>1</resolution>
               <min_angle>-3.14159</min_angle>
